File: pico_psu_mount.sch (KiCad schematic (older format))
At the start: 3 parts, among them J1 Conn_01x02, U1 DreamcastPower, U2 atx_24pin

Commit message: fixed: PicoPSU does not turns off properly, when no load is present on the 12V rail
Parts:
- added 10k1: R_Small, Resistors_SMD:R_0805_HandSoldering, symbol Device:R_Small
Connections:
- wire segments 41 -> 44
Changed lines of the file:
@@
 	8500 3300 8150 3300
 Wire Wire Line
-	6600 4100 8500 4100
+	6600 4100 7600 4100
 Wire Wire Line
 	6550 2000 8350 2000
@@
 	8350 2000 8350 2600
 Connection ~ 8350 2600
+$Comp
+L Device:R_Small 10k1
+U 1 1 5C0F1DC1
+P 7600 4250
+F 0 "10k1" H 7659 4296 50  0000 L CNN
+F 1 "R_Small" H 7659 4205 50  0000 L CNN
+F 2 "Resistors_SMD:R_0805_HandSoldering" H 7600 4250 50  0001 C CNN
+F 3 "~" H 7600 4250 50  0001 C CNN
+	1    7600 4250
+	1    0    0    -1
+$EndComp
+$Comp
+L power:GND #PWR0101
+U 1 1 5C0F1E4E
+P 7600 4400
+F 0 "#PWR0101" H 7600 4150 50  0001 C CNN
+F 1 "GND" H 7605 4227 50  0000 C CNN
+F 2 "" H 7600 4400 50  0001 C CNN
+F 3 "" H 7600 4400 50  0001 C CNN
+	1    7600 4400
+	1    0    0    -1
+$EndComp
+Wire Wire Line
+	7600 4150 7600 4100
+Connection ~ 7600 4100
+Wire Wire Line
+	7600 4100 8500 4100
+Wire Wire Line
+	7600 4400 7600 4350
 $EndSCHEMATC
